File: gaszähler.brd (EAGLE design)
At the start: 23.5 x 13.6 mm, 19 parts, among them IC1 LM358D

Commit message: adding images
Parts:
- removed D1: BPX65, opto-trans-siemens:BPX65
- removed LED1: (no value), led:LED5MM
- removed R4: 47, rcl:0207/10
- added GND_G, VCC_G: TPSQTP20SQ, testpad:TP20SQ
- added U$1: CNY70, cny70:4
- R1, R2, R3: device rcl:0207/10 -> rcl:R0805
- moved T1 77.7 mm to (43.2, 6.35), turned to 90 degrees
- moved R2 73.5 mm to (38.1, 3.81), turned to 180 degrees
- moved R3 62.5 mm to (38.1, 6.35), turned to 180 degrees
- moved R1 59.9 mm to (38.1, 8.89), turned to 180 degrees
- renumbered TP1 to SIGNAL, TP2 to GND, TP3 to VCC, TP4 to S0_SIG, TP5 to S0_GND
Connections:
- removed net +24V: D1.A, LED1.A, R3.2
- removed net N$12: R4.2
- removed net N$4: R2.1, R4.1, T1.E
- new net GND_G: GND_G.TP, R2.1, T1.E
- new net N$14: R3.2, U$1.A, U$1.C, VCC_G.TP
- net N$2: now also U$1.K; no longer LED1.K
- net N$3: now also U$1.E; no longer D1.K
Routing:
- net N$14: track 0.00 -> 29.4 mm
- net GND_G: track 0.00 -> 10.8 mm
- net N$3: track 0.00 -> 8.99 mm
- net N$6: track 0.00 -> 5.89 mm
- net N$2: track 0.00 -> 4.66 mm
- net N$7: track 0.00 -> 3.03 mm
- added copper zone on layer 1, net GND_G
Other:
- board size 23.5 x 13.6 mm -> 49.5 x 13.6 mm
